File: SODK-SMIT-No_Reflect_v2.0.kicad_pcb (KiCad board)
At the start: 2 copper layers, 157 parts, among them J1 REFLECT, J2 Conn_01x04, J3 Conn_01x04, J4 Conn_01x04, J5 Conn_01x04, J6 USB_OTG, Q1 BSS138, Q2 BSS138, Q3 2N3905, Q4 2N3904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

Commit message: 123
Parts:
- removed 2LM5IN2, LM33OUT1: CP1, Capacitors_THT:CP_Radial_D5.0mm_P2.00mm
- removed ENLM33: Conn_01x02, Pin_Headers:Pin_Header_Straight_1x02_Pitch2.54mm
- removed LM33IN1: D, Diodes_SMD:D_1206
- removed LM33IN2, LM33LEDR1: R, Resistors_SMD:R_0805
- removed LM33LED1: LED, LEDs:LED_0805
- removed U5: LM1117-3.3, TO_SOT_Packages_SMD:SOT-223-3_TabPin2
- added 1k1: R, Resistors_SMD:R_0805, F.Cu at (92.0, 60.0)
- added AE1: Antenna_Shield, Connectors:SMB_Straight, F.Cu at (94.0, 36.0)
- added C5: C, Capacitors_SMD:C_0805, F.Cu at (66.3, 34.6)
- added C6: C, Capacitors_SMD:C_0805, F.Cu at (72.0, 34.8)
- added C7: C, Capacitors_SMD:C_0805, F.Cu at (73.8, 34.8)
- added C8: CP1, Capacitors_THT:CP_Radial_D5.0mm_P2.00mm, F.Cu at (74.3, 30.5)
- added D5817: D, Diodes_THT:D_DO-41_SOD81_P7.62mm_Horizontal, F.Cu at (89.5, 60.0)
- added ENGPS1: Conn_01x02, Pin_Headers:Pin_Header_Straight_1x02_Pitch2.54mm, F.Cu at (69.3, 31.3)
- added GPS1: MOUDLE-GPS-NEO-6M(24P-16X12.2MM), MOUDLE-GPS-NEO-6M_24P-16X12.2MM_:GPS24P-SMD-1.1-16X12.2MM, F.Cu at (87.5, 49.5)
- added GPS33LED1: LED, LEDs:LED_0805, F.Cu at (75.6, 34.9)
- added GPSINLED1: LED, LEDs:LED_0805, F.Cu at (98.0, 55.5)
- added GPSINLEDR1: R, Resistors_SMD:R_0805, F.Cu at (96.0, 55.5)
- added GPSLEDR1: R, Resistors_SMD:R_0805, B.Cu at (75.7, 34.9)
- added GPSMEM1: 24AA32AT-I/MS, 24AA32AT-I_MS:SOP65P490X110-8N, B.Cu at (87.5, 52.5)
- added LGPS1: L, Inductors_SMD:L_1812, F.Cu at (85.0, 38.5)
- added MIC33: MIC5218-3.3, TO_SOT_Packages_SMD:SOT-23-5, F.Cu at (69.1, 34.6)
- added PCB_ANT1: Antenna, Measurement_Points:Test_Point_Keystone_5015_Micro-Minature, F.Cu at (31.0, 2.54)
- added RGPS1: R, Resistors_SMD:R_0805, F.Cu at (96.8, 44.4)
- added RX1R1: R, Resistors_SMD:R_0805, F.Cu at (52.9, 60.3)
- added TX1R1: R, Resistors_SMD:R_0805, F.Cu at (54.5, 60.3)
- 100n4.1, 100nV1, 100nV2, 100nV3, 10K3, 10K4, 1MC1, 1u4.1, 1uF2, 22pC1, 22pC2, 22pF1, 22pF2, 2LMIN2, 470r4.1, 4k7I1, 4k7I2, C1, C104, C2, C3, C4, D2, LMIN2: moved to B.Cu
- SIMCARD1: footprint Sockets:ADSP2100 -> conn-sim:ICC-313
- moved C101_1 189.9 mm to (13.6, 22.0), turned to 270 degrees
- moved 22pF2 188.5 mm to (26.2, 16.7), turned to 180 degrees
- moved USB1 187.7 mm to (19.7, 10.6), turned to 90 degrees
- moved C101 185.5 mm to (31.4, 4.98)
- moved 22pF1 185.0 mm to (26.2, 18.2)
- moved 4k7NETSIM1 180.6 mm to (9.49, 28.6)
- moved 33pSIM1 172.6 mm to (5.38, 42.0)
- moved USB_PWR1 172.6 mm to (10.9, 4.15), turned to 90 degrees
- moved C101_2 171.1 mm to (18.9, 22.0), turned to 270 degrees
- moved CbSIM1 171.1 mm to (5.36, 40.3)
- moved 5M+2 169.9 mm to (21.0, 94.5)
- moved 100nF1 168.6 mm to (38.2, 11.4)
- moved 10pSIM1 168.3 mm to (5.39, 43.8)
- moved Q4 167.9 mm to (5.27, 29.3), turned to 90 degrees
- moved RX0 167.2 mm to (38.5, 44.0)
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Connections:
- 10kS/A6 pad 2: TX0 -> TX1
- 10kS/A8 pad 2: RX0 -> RX1
- 4.1LEDR1 pad 2: Net-(4.1LEDR1-Pad2) -> VBAT
- Q5 pad 3: TX0 -> TX1
- Q6 pad 3: RX0 -> RX1
- U1 pad 7: Net-(U1-Pad7) -> ENSIM800
- U1 pad 78: Net-(U1-Pad78) -> ON4.1
- U9 pad 39: PWEKEY -> PWRKEY
Routing:
- net +5V: track 0.00 -> 523.0 mm, vias 0 -> 18
- net GND: track 0.00 -> 359.2 mm, vias 0 -> 28
- net VBAT: track 0.00 -> 148.7 mm, vias 0 -> 4
- net +3V3: track 0.00 -> 90.4 mm, vias 0 -> 1
- net LINE1: track 0.00 -> 80.1 mm
- net A4_EXT: track 0.00 -> 77.5 mm
- net RESET: track 0.00 -> 76.1 mm, vias 0 -> 5
- net LINE2: track 0.00 -> 75.1 mm, vias 0 -> 1
- net LINE3: track 0.00 -> 69.2 mm, vias 0 -> 1
- net A3_EXT: track 0.00 -> 68.7 mm
- net T1_EXT: track 0.00 -> 67.7 mm, vias 0 -> 1
- net LINE4: track 0.00 -> 61.7 mm, vias 0 -> 1
- net A1_EXT: track 0.00 -> 61.4 mm
- net A2_EXT: track 0.00 -> 56.7 mm
- net LED_IN: track 0.00 -> 55.6 mm, vias 0 -> 2
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- added copper zone on B.Cu, net GND
- added copper zone on F.Cu, net GND
Other:
- board outline added: 100 x 100 mm
