File: SODK-SMIT-No_Reflect_v2.0.sch (KiCad schematic (older format))
At the start: 82 parts

Commit message: 123
Parts:
- added 100nF (x2), 1uF (x2), 22pF (x2), C101 (x4), C104, C? (x4): C, symbol C
- added 10K (x4), 4.7K (x2), 4.7K? (x3), 5M+, 5M+? (x3), L1R, L2R, L3R, L4R, LED_IN_R, R101_0Om, R?: R, symbol R
- added 12Mhz: Crystal, symbol Crystal
- added ADS1115_LED, L1Led, L2Led, L3Led, L4Led, USB_PWR: LED, symbol LED
- added EXT_ANT: Antenna_Shield, symbol Antenna_Shield
- added IN1, IN2, IN3, IN4, IN5: WS2812B, WS2812B, symbol WS2812B
- added J?: USB_OTG, symbol USB_OTG
- added J? (x4): Conn_01x04, symbol Conn_01x04
- added L1, L2, L3, L4: Conn_01x03, symbol Conn_01x03
- added MMZ2012Y152B (x2): Ferrite_Bead, symbol Ferrite_Bead
- added PCB_ANT: Antenna, symbol Antenna
- added Q?: 2N3905, TO_SOT_Packages_THT:TO-92_Molded_Narrow, symbol 2N3905
- added RTC: CP, symbol CP
- added U?: SIM800C, LCC110P1570X1760X250-42N, symbol SIM800C
- added U?: AN91445, symbol AN91445
- added U?: ADS1115, MSOP10, symbol ADS1115
- added U?: CH340, SO16, symbol CH340
- added USB: D, symbol D
Connections:
- net +5V: now also 1uF.1, 4.7K.1, 4.7K.2, 4.7K?.2, 4.7K?.2, 4.7K?.2, 5M+.2, 5M+?.2, 5M+?.2, 5M+?.2, C104.1, C?.1, C?.1, C?.1, C?.1, IN1.1 (VDD), IN2.1 (VDD), IN3.1 (VDD), IN4.1 (VDD), IN5.1 (VDD), J?.1 (Pin_1), J?.1 (Pin_1), J?.1 (Pin_1), J?.1 (Pin_1), MMZ2012Y152B.1, Q?.3 (C), U?.16 (VCC), USB.1 (K)
- net GND: now also 100nF.2, 10K.1, 1uF.2, 1uF.2, 22pF.1, 22pF.2, ADS1115_LED.1 (K), C101.2, C101.2, C101.2, C101.2, C104.2, C?.2, C?.2, C?.2, C?.2, EXT_ANT.2 (Shield), IN1.3 (VSS), IN2.3 (VSS), IN3.3 (VSS), IN4.3 (VSS), IN5.3 (VSS), J?.4 (Pin_4), J?.4 (Pin_4), J?.4 (Pin_4), J?.4 (Pin_4), J?.5 (GND), L1.3 (Pin_3), L1Led.1 (K), L1R.1, L2.3 (Pin_3), L2Led.1 (K), L2R.1, L3.3 (Pin_3), L3Led.1 (K), L3R.1, L4.3 (Pin_3), L4Led.1 (K), L4R.1, MMZ2012Y152B.1, MMZ2012Y152B.2, Q?.1 (E), RTC.2, U?.1 (GND), U?.13 (GND), U?.19 (GND), U?.2 (GND), U?.21 (GND), U?.27 (GND), U?.3 (VSS), U?.30 (GND), U?.31 (GND), U?.33 (GND), U?.36 (GND), U?.37 (GND), U?.8 (GND), USB_PWR.1 (K)
- net NETLIGHT: now also U?.41 (NETLIGHT)
- net RESET: now also 100nF.1
- net RX0: now also U?.2 (TXD)
- net RXSIM: now also U?.2 (UART1_RXD)
- net SCL: now also 10K.2, U?.10 (SCL)
- net SDA: now also 10K.2, U?.9 (SDA)
- net SIMCLK: now also U?.16 (SIM_CLK)
- net SIMDATA: now also U?.15 (SIM_DATA)
- net SIMDET: now also U?.14 (SIM_DET)
- net SIMRST: now also U?.17 (SIM_RST)
- net SIMVDD: now also U?.18 (SIM_VDD)
- net TX0: now also U?.3 (RXD)
- net TXSIM: now also U?.1 (UART1_TXD)
- net VBAT: now also U?.34 (VBAT), U?.35 (VBAT)
- net T_INT: now reaches U?.25 ((PCINT6/OC1B)PB6)
- net T_INT: now also 4.7K.2, Q?.2 (B)
- net LED_IN: now reaches U?.26 ((PCINT7/OC0A/OC1C)PB7)
- net LED_IN: now also LED_IN_R.1
- net LINE1: now reaches U?.53 ((A8)PC0)
- net LINE1: now also L1.1 (Pin_1)
- net LINE2: now reaches U?.54 ((A9)PC1)
- net LINE2: now also L2.1 (Pin_1)
- net LINE3: now reaches U?.55 ((A10)PC2)
- net LINE3: now also L3.1 (Pin_1)
- net LINE4: now reaches U?.56 ((A11)PC3)
- net LINE4: now also L4.1 (Pin_1)
- net T1_EXT: now reaches U?.57 ((A12)PC4)
- net T1_EXT: now also 4.7K.1, J?.2 (Pin_2)
- net T2_EXT: now reaches U?.58 ((A13)PC5)
- net T2_EXT: now also 4.7K?.1, J?.2 (Pin_2)
- net T3_EXT: now reaches U?.59 ((A14)PC6)
- net T3_EXT: now also 4.7K?.1, J?.2 (Pin_2)
- net T4_EXT: now reaches U?.60 ((A15)PC7)
- net T4_EXT: now also 4.7K?.1, J?.2 (Pin_2)
- net A4_EXT: now reaches U?.82 (PK7(ADC15/PCINT23))
- net A4_EXT: now also J?.3 (Pin_3)
- net A3_EXT: now reaches U?.83 (PK6(ADC14/PCINT22))
- net A3_EXT: now also J?.3 (Pin_3)
- net A2_EXT: now reaches U?.84 (PK5(ADC13/PCINT21))
- net A2_EXT: now also J?.3 (Pin_3)
- net A1_EXT: now reaches U?.85 (PK4(ADC12/PCINT20))
- net A1_EXT: now also J?.3 (Pin_3)
- new net: C101.1, R?.1, U?.20 (BT_ANT)
- new net: RTC.1, U?.28 (VRTC)
- new net: C101.1, EXT_ANT.1 (A), R101_0Om.1, U?.32 (GSM_ANT)
- new net: C101.1, PCB_ANT.1 (A), R101_0Om.2
- new net: C101.1, R?.2, U?.1 (SIG)
- new net: 10K.2, U?.1 (ADDR)
- new net: 100nF.2, U?.13 (DTR#)
- new net: 100nF.1, U?.4 (V3)
- new net: J?.3 (D+), U?.5 (UD+)
- new net: J?.2 (D-), U?.6 (UD)
- new net: 12Mhz.1, 22pF.2, U?.7 (XI)
- new net: 12Mhz.2, 22pF.1, U?.8 (XO)
- new net: J?.1 (VBUS), USB.2 (A), USB_PWR.2 (A)
- new net: L1Led.2 (A), L1R.2
- new net: L2Led.2 (A), L2R.2
- new net: L3Led.2 (A), L3R.2
- new net: L4Led.2 (A), L4R.2
- new net: IN1.2 (DOUT), IN2.4 (DIN)
- new net: IN1.4 (DIN), LED_IN_R.2
- new net: IN2.2 (DOUT), IN3.4 (DIN)
- new net: IN3.2 (DOUT), IN4.4 (DIN)
- new net: IN4.2 (DOUT), IN5.4 (DIN)
- new net +5VP: 10K.1, 10K.1, 10K.1, 1uF.1, ADS1115_LED.2 (A), MMZ2012Y152B.2, U?.8 (VDD)
- new net AIN0: 5M+.1, L1.2 (Pin_2), U?.4 (AIN0)
- new net AIN1: 5M+?.1, L2.2 (Pin_2), U?.5 (AIN1)
- new net AIN2: 5M+?.1, L3.2 (Pin_2), U?.6 (AIN2)
- new net AIN3: 5M+?.1, L4.2 (Pin_2), U?.7 (AIN3)
- new net DRDY: 10K.2, U?.2 (ALERT/RDY)
- new net PWEKEY: U?.39 (PWRKEY)
- new net STATUS: U?.42 (STATUS)
Other:
- note added: "ADS1115\n"
- note added: "CH340G USB\n"
- note added: "I2C Addr = 1001000"
- note added: "SIM800C\n"

Commit message: 123
Parts:
- added 10kS/A? (x4), R_LED_REFLECT: R, symbol R
- added J?: REFLECT, symbol Conn_01x06
- added LED_REFLECT: LED, symbol LED
- added Q? (x2): BSS138, TO_SOT_Packages_SMD:SOT-23, symbol BSS138
Connections:
- net +5V: now also 10kS/A?.1, 10kS/A?.1, J?.1 (Pin_1)
- net GND: now also J?.6 (Pin_6), LED_REFLECT.1 (K)
- net RX2: now also 10kS/A?.2, Q?.3 (D)
- net TX2: now also 10kS/A?.2, Q?.3 (D)
- new net: J?.5 (Pin_5), R_LED_REFLECT.1
- new net: LED_REFLECT.2 (A), R_LED_REFLECT.2
- new net RXREF: 10kS/A?.2, J?.3 (Pin_3), Q?.2 (S)
- new net TXREF: 10kS/A?.2, J?.4 (Pin_4), Q?.2 (S)
- new net VREF: 10kS/A?.1, 10kS/A?.1, J?.2 (Pin_2), Q?.1 (G), Q?.1 (G)
Other:
- note added: "REFLECT-INPUT/OUTPUT\n"
Changed lines of the file:
@@
 Text GLabel 5150 3800 2    60   Input ~ 0
 T_INT
+$Comp
+L BSS138 Q?
+U 1 1 5A8EFF44
+P 8225 2750
+F 0 "Q?" H 8425 2825 50  0000 L CNN
+F 1 "BSS138" H 8425 2750 50  0000 L CNN
+F 2 "TO_SOT_Packages_SMD:SOT-23" H 8425 2675 50  0001 L CIN
+F 3 "" H 8225 2750 50  0001 L CNN
+	1    8225 2750
+	0    1    1    0
+$EndComp
+$Comp
+L +5V #PWR?
+U 1 1 5A8EFF4A
+P 8425 2550
+F 0 "#PWR?" H 8425 2400 50  0001 C CNN
+F 1 "+5V" H 8425 2690 50  0000 C CNN
+F 2 "" H 8425 2550 50  0001 C CNN
+F 3 "" H 8425 2550 50  0001 C CNN
+	1    8425 2550
+	1    0    0    -1
+$EndComp
+$Comp
+L R 10kS/A?
+U 1 1 5A8EFF50
+P 8425 2700
+F 0 "10kS/A?" V 8505 2700 50  0000 C CNN
+F 1 "R" V 8425 2700 50  0000 C CNN
+F 2 "" V 8355 2700 50  0001 C CNN
+F 3 "" H 8425 2700 50  0001 C CNN
+	1    8425 2700
+	1    0    0    -1
+$EndComp
+Text GLabel 8025 2550 1    60   Input ~ 0
+VREF
+$Comp
+L R 10kS/A?
+U 1 1 5A8EFF57
+P 8025 2700
+F 0 "10kS/A?" V 8105 2700 50  0000 C CNN
+F 1 "R" V 8025 2700 50  0000 C CNN
+F 2 "" V 7955 2700 50  0001 C CNN
+F 3 "" H 8025 2700 50  0001 C CNN
+	1    8025 2700
+	1    0    0    -1
+$EndComp
+Text GLabel 8425 2850 2    60   Input ~ 0
+RX2
+Text GLabel 8025 2850 0    60   Input ~ 0
+TXREF
+Wire Wire Line
+	8225 2550 8025 2550
+$Comp
+L BSS138 Q?
+U 1 1 5A8F0766
+P 7175 2750
+F 0 "Q?" H 7375 2825 50  0000 L CNN
+F 1 "BSS138" H 7375 2750 50  0000 L CNN
+F 2 "TO_SOT_Packages_SMD:SOT-23" H 7375 2675 50  0001 L CIN
+F 3 "" H 7175 2750 50  0001 L CNN
+	1    7175 2750
+	0    1    1    0
+$EndComp
+$Comp
+L +5V #PWR?
+U 1 1 5A8F076C
+P 7375 2550
+F 0 "#PWR?" H 7375 2400 50  0001 C CNN
+F 1 "+5V" H 7375 2690 50  0000 C CNN
+F 2 "" H 7375 2550 50  0001 C CNN
+F 3 "" H 7375 2550 50  0001 C CNN
+	1    7375 2550
+	1    0    0    -1
+$EndComp
+$Comp
+L R 10kS/A?
+U 1 1 5A8F0772
+P 7375 2700
+F 0 "10kS/A?" V 7455 2700 50  0000 C CNN
+F 1 "R" V 7375 2700 50  0000 C CNN
+F 2 "" V 7305 2700 50  0001 C CNN
+F 3 "" H 7375 2700 50  0001 C CNN
+	1    7375 2700
+	1    0    0    -1
+$EndComp
+Text GLabel 6975 2550 1    60   Input ~ 0
+VREF
+$Comp
+L R 10kS/A?
+U 1 1 5A8F0779
+P 6975 2700
+F 0 "10kS/A?" V 7055 2700 50  0000 C CNN
+F 1 "R" V 6975 2700 50  0000 C CNN
+F 2 "" V 6905 2700 50  0001 C CNN
+F 3 "" H 6975 2700 50  0001 C CNN
+	1    6975 2700
+	1    0    0    -1
+$EndComp
+Text GLabel 7375 2850 2    60   Input ~ 0
+TX2
+Text GLabel 6975 2850 0    60   Input ~ 0
+RXREF
+Wire Wire Line
+	7175 2550 6975 2550
+$Comp
+L Conn_01x06 J?
+U 1 1 5A8F1000
+P 7675 3025
+F 0 "J?" H 7675 3325 50  0000 C CNN
+F 1 "REFLECT" H 7675 2625 50  0000 C CNN
+F 2 "" H 7675 3025 50  0001 C CNN
+F 3 "" H 7675 3025 50  0001 C CNN
+	1    7675 3025
+	0    -1   -1   0
+$EndComp
+$Comp
+L +5V #PWR?
+U 1 1 5A8F1AEC
+P 7475 3225
+F 0 "#PWR?" H 7475 3075 50  0001 C CNN
+F 1 "+5V" H 7475 3365 50  0000 C CNN
+F 2 "" H 7475 3225 50  0001 C CNN
+F 3 "" H 7475 3225 50  0001 C CNN
+	1    7475 3225
+	-1   0    0    1
+$EndComp
+Text GLabel 7575 3225 3    60   Input ~ 0
+VREF
+Text GLabel 7675 3225 3    60   Input ~ 0
+RXREF
+Text GLabel 7775 3225 3    60   Input ~ 0
+TXREF
+$Comp
+L GND #PWR?
+U 1 1 5A8F21B7
+P 7975 3225
+F 0 "#PWR?" H 7975 2975 50  0001 C CNN
+F 1 "GND" H 7975 3075 50  0000 C CNN
+F 2 "" H 7975 3225 50  0001 C CNN
+F 3 "" H 7975 3225 50  0001 C CNN
+	1    7975 3225
+	1    0    0    -1
+$EndComp
+$Comp
+L LED LED_REFLECT
+U 1 1 5A8F2303
+P 8225 3450
+F 0 "LED_REFLECT" H 8225 3550 50  0000 C CNN
+F 1 "LED" H 8225 3350 50  0000 C CNN
+F 2 "" H 8225 3450 50  0001 C CNN
+F 3 "" H 8225 3450 50  0001 C CNN
+	1    8225 3450
+	-1   0    0    1
+$EndComp
+$Comp
+L R R_LED_REFLECT
+U 1 1 5A8F24A0
+P 7875 3375
+F 0 "R_LED_REFLECT" V 7955 3375 50  0000 C CNN
+F 1 "R" V 7875 3375 50  0000 C CNN
+F 2 "" V 7805 3375 50  0001 C CNN
+F 3 "" H 7875 3375 50  0001 C CNN
+	1    7875 3375
+	1    0    0    -1
+$EndComp
+Wire Wire Line
+	7875 3525 8025 3525
+Wire Wire Line
+	8025 3525 8025 3450
+Wire Wire Line
+	8025 3450 8075 3450
+$Comp
+L GND #PWR?
+U 1 1 5A8F28CE
+P 8375 3450
+F 0 "#PWR?" H 8375 3200 50  0001 C CNN
+F 1 "GND" H 8375 3300 50  0000 C CNN
+F 2 "" H 8375 3450 50  0001 C CNN
+F 3 "" H 8375 3450 50  0001 C CNN
+	1    8375 3450
+	0    -1   -1   0
+$EndComp
+Wire Notes Line
+	5950 2000 5950 3600
+Wire Notes Line
+	5950 3600 7050 3600
+Text Notes 6125 2175 0    60   ~ 0
+REFLECT-INPUT/OUTPUT\n
 $EndSCHEMATC

Commit message: 123
Parts:
- 100k4.1, 43k4.1, 470r4.1, RX0, RX2, RX3, TX0, TX2, TX3: footprint (none) -> Resistors_SMD:R_0805
- 100n4.1, 1u4.1, C101, C104: footprint (none) -> Capacitors_SMD:C_0805
- 100nF1, 100nF2: renamed from 100nF; footprint (none) -> Capacitors_SMD:C_0805
- 100nSIMCARD1: renamed from 100nSIMCARD; footprint (none) -> Capacitors_SMD:C_0805
- 100nV1, 100nV2, 100nV3: renamed from 100nV; footprint (none) -> Capacitors_SMD:C_0805
- 100u4.1, 330u4.1: footprint (none) -> Capacitors_THT:CP_Radial_D5.0mm_P2.00mm
- 10K1, 10K2, 10K3, 10K4: renamed from 10K; footprint (none) -> Resistors_SMD:R_0805
- 10kRST1: renamed from 10kRST; footprint (none) -> Resistors_SMD:R_0805
- 10kS/A1, 10kS/A2, 10kS/A3, 10kS/A4, 10kS/A7, 10kS/A8: renamed from 10kS/A?; footprint (none) -> Resistors_SMD:R_0805
- 10kS/A5, 10kS/A6: renamed from 10kS/A; footprint (none) -> Resistors_SMD:R_0805
- 10pSIM1: renamed from 10pSIM; footprint (none) -> Capacitors_SMD:C_0805
- 12Mhz1: renamed from 12Mhz; footprint (none) -> Crystals:Crystal_HC49-U_Vertical
- 16MHZ1: renamed from 16MHZ; footprint (none) -> Crystals:Crystal_HC49-U_Vertical
- 1MC1: renamed from 1MC; footprint (none) -> Resistors_SMD:R_0805
- 1uF1, 1uF2: renamed from 1uF; footprint (none) -> Capacitors_SMD:C_0805
- 22pC1, 22pC2: renamed from 22pC; footprint (none) -> Capacitors_SMD:C_0805
- 22pF1, 22pF2: renamed from 22pF; footprint (none) -> Capacitors_SMD:C_0805
- 22pRST1: renamed from 22pRST; footprint (none) -> Capacitors_SMD:C_0805
- 22pSIMCARD1: renamed from 22pSIMCARD; footprint (none) -> Capacitors_SMD:C_0805
- 2LM5IN1: renamed from 2LM5IN; footprint (none) -> Capacitors_THT:CP_Radial_D5.0mm_P2.00mm
- 2LM5IN2: renamed from 2LM5IN?; footprint (none) -> Capacitors_THT:CP_Radial_D5.0mm_P2.00mm
- 2LM5OUT1: renamed from 2LM5OUT; footprint (none) -> Capacitors_THT:CP_Radial_D5.0mm_P2.00mm
- 2LMIN1: renamed from 2LMIN; footprint (none) -> Diodes_SMD:D_1206
- 2LMIN2: renamed from 2LMIN; footprint (none) -> Resistors_SMD:R_0402
- 2LMLED1: renamed from 2LMLED; footprint (none) -> LEDs:LED_0805
- 2LMLEDR1: renamed from 2LMLEDR; footprint (none) -> Resistors_SMD:R_0805
- 33pSIM1: renamed from 33pSIM; footprint (none) -> Capacitors_SMD:C_0805
- 4.1LEDR1: renamed from 4.1LEDR; footprint (none) -> Resistors_SMD:R_0805
- 4.7K1, 4.7K5: renamed from 4.7K; footprint (none) -> Resistors_SMD:R_0805
- 4.7K2, 4.7K3, 4.7K4: renamed from 4.7K?; footprint (none) -> Resistors_SMD:R_0805
- 47kNETSIM1: renamed from 47kNETSIM; footprint (none) -> Resistors_SMD:R_0805
- 4k7ENSIM1, 4k7ENSIM2: renamed from 4k7ENSIM; footprint (none) -> Resistors_SMD:R_0805
- 4k7I1, 4k7I2: renamed from 4k7I; footprint (none) -> Resistors_SMD:R_0805
- 4k7NETSIM1: renamed from 4k7NETSIM; footprint (none) -> Resistors_SMD:R_0805
- 5.1v500mWSIM1: renamed from 5.1v500mWSIM; footprint (none) -> Diodes_SMD:D_SOD-123
- 51rSIMCARD1, 51rSIMCARD2, 51rSIMCARD3: renamed from 51rSIMCARD; footprint (none) -> Resistors_SMD:R_0805
- 5M+1: renamed from 5M+; footprint (none) -> Resistors_SMD:R_0805
- 5M+2, 5M+3, 5M+4: renamed from 5M+?; footprint (none) -> Resistors_SMD:R_0805
- ADS1115_LED1: renamed from ADS1115_LED; footprint (none) -> LEDs:LED_0805
- AREF100n1: renamed from AREF100n; footprint (none) -> Capacitors_SMD:C_0805
- C1, C2, C3, C4: renamed from C?; footprint (none) -> Capacitors_SMD:C_0805
- C101_1, C101_2, C101_3: renamed from C101; footprint (none) -> Capacitors_SMD:C_0805
- CaSIM1: renamed from CaSIM; footprint (none) -> Capacitors_THT:CP_Radial_D5.0mm_P2.00mm
- CbSIM1: renamed from CbSIM; footprint (none) -> Capacitors_SMD:C_0805
- D1: renamed from D?; footprint (none) -> LEDs:LED_0805
- D2: renamed from D?; footprint (none) -> TO_SOT_Packages_SMD:SOT-363_SC-70-6_Handsoldering
- EN2LM5, ENLM33, ENLM5: footprint (none) -> Pin_Headers:Pin_Header_Straight_1x02_Pitch2.54mm
- EXT_ANT1: renamed from EXT_ANT; footprint (none) -> Connectors:SMA_THT_Jack_Straight
- ICSP1: renamed from ICSP; footprint (none) -> Pin_Headers:Pin_Header_Straight_1x06_Pitch2.00mm
- IN1, IN2, IN3, IN4, IN5: footprint WS2812B -> WS2812B:WS2812B
- J1: renamed from J?; footprint (none) -> Pin_Headers:Pin_Header_Straight_1x06_Pitch2.00mm
- J2, J3, J4, J5: renamed from J?; footprint (none) -> Pin_Headers:Pin_Header_Straight_1x04_Pitch2.00mm
- J6: renamed from J?; footprint (none) -> Connectors_USB:USB_Micro-B_Wuerth-629105150521
- L1, L2, L3, L4: footprint (none) -> Pin_Headers:Pin_Header_Straight_1x03_Pitch2.00mm
- L1Led1: renamed from L1Led; footprint (none) -> LEDs:LED_0805
- L1R1: renamed from L1R; footprint (none) -> Resistors_SMD:R_0805
- L2Led1: renamed from L2Led; footprint (none) -> LEDs:LED_0805
- L2R1: renamed from L2R; footprint (none) -> Resistors_SMD:R_0805
- L3Led1: renamed from L3Led; footprint (none) -> LEDs:LED_0805
- L3R1: renamed from L3R; footprint (none) -> Resistors_SMD:R_0805
- L4Led1: renamed from L4Led; footprint (none) -> LEDs:LED_0805
- L4R1: renamed from L4R; footprint (none) -> Resistors_SMD:R_0805
- LED_IN_R1: renamed from LED_IN_R; footprint (none) -> Resistors_SMD:R_0805
- LED_REFLECT1: renamed from LED_REFLECT; footprint (none) -> LEDs:LED_0805
- LM33IN1: renamed from LM33IN; footprint (none) -> Diodes_SMD:D_1206
- LM33IN2: renamed from LM33IN; footprint (none) -> Resistors_SMD:R_0805
- LM33LED1: renamed from LM33LED; footprint (none) -> LEDs:LED_0805
- LM33LEDR1: renamed from LM33LEDR; footprint (none) -> Resistors_SMD:R_0805
- LM33OUT1: renamed from LM33OUT; footprint (none) -> Capacitors_THT:CP_Radial_D5.0mm_P2.00mm
- LM5IN1: renamed from LM5IN; footprint (none) -> Capacitors_THT:CP_Radial_D5.0mm_P2.00mm
- LM5OUT1: renamed from LM5OUT; footprint (none) -> Capacitors_THT:CP_Radial_D5.0mm_P2.00mm
- LMIN1: renamed from LMIN; footprint (none) -> Diodes_SMD:D_1206
- LMIN2: renamed from LMIN; footprint (none) -> Resistors_SMD:R_0805
- LMLED1: renamed from LMLED; footprint (none) -> LEDs:LED_0805
- LMLEDR1: renamed from LMLEDR; footprint (none) -> Resistors_SMD:R_0805
- MMZ2012Y152B1, MMZ2012Y152B2: renamed from MMZ2012Y152B; footprint (none) -> Inductors_SMD:L_0805
- NETLIGHTSIM1: renamed from NETLIGHTSIM; footprint (none) -> LEDs:LED_0805
- R1: renamed from R?; footprint (none) -> Resistors_SMD:R_0805
- R101_0Om1: renamed from R101_0Om; footprint (none) -> Resistors_SMD:R_0805
- RGB1: renamed from RGB; footprint (none) -> Resistors_SMD:R_0805
- RTC1: renamed from RTC; footprint (none) -> Capacitors_THT:CP_Radial_D5.0mm_P2.00mm
- RVB1: renamed from RVB; footprint (none) -> Resistors_SMD:R_0805
- R_LED_REFLECT1: renamed from R_LED_REFLECT; footprint (none) -> Resistors_SMD:R_0805
- SIMCARD1: renamed from SIMCARD; footprint (none) -> Sockets:ADSP2100
- SW1: renamed from SW?; footprint (none) -> Buttons_Switches_SMD:SW_SPST_FSMSM
- U1: renamed from U?; footprint TQFP100 -> Housings_QFP:TQFP-100_14x14mm_Pitch0.5mm
- U2, U3, U5: renamed from U?; footprint (none) -> TO_SOT_Packages_SMD:SOT-223-3_TabPin2
- U4: renamed from U?; footprint MSOP10 -> ADS1115:MSOP10
- U6: renamed from U?; footprint (none) -> TO_SOT_Packages_THT:TO-220-5_Horizontal
- U7: renamed from U?; footprint (none) -> MyAntennas:AN91445
- U8: renamed from U?; footprint SO16 -> CH340:SO16
- U9: renamed from U?; footprint LCC110P1570X1760X250-42N -> SIM800C:LCC110P1570X1760X250-42N
- USB1: renamed from USB; footprint (none) -> Diodes_SMD:D_1206
- USB_PWR1: renamed from USB_PWR; footprint (none) -> LEDs:LED_0805
- gave numbers to parts that had none: 6
- renumbered ENSIM to ENSIM1, PCB_ANT to PCB_ANT1

Commit message: 123
Parts:
- removed 2LM5IN2, LM33OUT1: CP1, Capacitors_THT:CP_Radial_D5.0mm_P2.00mm, symbol CP1
- removed ENLM33: Conn_01x02, Pin_Headers:Pin_Header_Straight_1x02_Pitch2.54mm, symbol Conn_01x02
- removed LM33IN1: D, Diodes_SMD:D_1206, symbol D
- removed LM33IN2, LM33LEDR1: R, Resistors_SMD:R_0805, symbol R
- removed LM33LED1: LED, LEDs:LED_0805, symbol LED
- removed U5: LM1117-3.3, TO_SOT_Packages_SMD:SOT-223-3_TabPin2, symbol LM1117-5.0
- added 1k1, GPSINLEDR1, GPSLEDR1, RGPS1, RX1R1, TX1R1: R, Resistors_SMD:R_0805, symbol R
- added AE1: Antenna_Shield, Connectors:SMB_Straight, symbol Antenna_Shield
- added C5, C6, C7: C, Capacitors_SMD:C_0805, symbol C
- added C8: CP1, Capacitors_THT:CP_Radial_D5.0mm_P2.00mm, symbol CP1
- added D5817: D, Diodes_THT:D_DO-41_SOD81_P7.62mm_Horizontal, symbol D
- added ENGPS1: Conn_01x02, Pin_Headers:Pin_Header_Straight_1x02_Pitch2.54mm, symbol Conn_01x02
- added GPS1: MOUDLE-GPS-NEO-6M(24P-16X12.2MM), MOUDLE-GPS-NEO-6M_24P-16X12.2MM_:GPS24P-SMD-1.1-16X12.2MM, symbol MOUDLE-GPS-NEO-6M(24P-16X12.2MM)
- added GPS33LED1, GPSINLED1: LED, LEDs:LED_0805, symbol LED
- added GPSMEM1: 24AA32AT-I/MS, 24AA32AT-I_MS:SOP65P490X110-8N, symbol 24AA32AT-I/MS
- added LGPS1: L, Inductors_SMD:L_1812, symbol L
- added MIC33: MIC5218-3.3, TO_SOT_Packages_SMD:SOT-23-5, symbol MIC5219-2.5
- PCB_ANT1: footprint (none) -> Measurement_Points:Test_Point_Keystone_5015_Micro-Minature
- SIMCARD1: footprint Sockets:ADSP2100 -> conn-sim:ICC-313
Connections:
- net PWEKEY is gone; now on net PWRKEY: U9.39 (PWRKEY)
- net +3V3: now also C6.1, C7.1, C8.1, D5817.2 (A), GPS1.23 (VCC), GPS33LED1.2 (A), GPSMEM1.8 (VCC), MIC33.5 (OUT)
- net +5V: now also ENGPS1.1 (Pin_1)
- net ENSIM800: now also U1.7 ((OC3C/INT5)PE5)
- net GND: now also AE1.2 (Shield), C5.2, C6.2, C7.2, C8.2, GPS1.10 (GND), GPS1.12 (GND2), GPS1.13 (GND3), GPS1.24 (GND4), GPSINLED1.1 (K), GPSLEDR1.2, GPSMEM1.1 (A0), GPSMEM1.2 (A1), GPSMEM1.3 (A2), GPSMEM1.4 (VSS), GPSMEM1.7 (WP), MIC33.2 (GND)
- net ON4.1: now also U1.78 ((AD0)PA0)
- net RX0: no longer 10kS/A8.2, Q6.3 (D)
- net RX3: now also GPS1.20 (TX)
- net TX0: no longer 10kS/A6.2, Q5.3 (D)
- net TX3: now also GPS1.21 (RX)
- net VBAT: now also 4.1LEDR1.2
- net at U1.45 ((RXD1/INT2)PD2): now also RX1R1.2
- net at U1.46 ((TXD1/INT3)PD3): now also TX1R1.2
- new net: C5.1, ENGPS1.2 (Pin_2), MIC33.1 (IN), MIC33.3 (EN)
- new net: GPS33LED1.1 (K), GPSLEDR1.1
- new net: AE1.1 (A), GPS1.11 (RFIN), LGPS1.2
- new net: GPS1.18 (SDA), GPSMEM1.5 (SDA)
- new net: GPS1.19 (SCL), GPSMEM1.6 (SCL)
- new net: 1k1.2, GPS1.22 (VB)
- new net: GPS1.3 (TP), GPSINLEDR1.1
- new net: GPS1.8 (NC3), GPS1.9 (VRF), RGPS1.1
- new net: GPSINLED1.2 (A), GPSINLEDR1.2
- new net: LGPS1.1, RGPS1.2
- new net: 1k1.1, D5817.1 (K)
- new net RX1: 10kS/A8.2, Q6.3 (D), RX1R1.1
- new net TX1: 10kS/A6.2, Q5.3 (D), TX1R1.1
Other:
- moved on the sheet: C101, C101_1, C101_2, C101_3, EXT_ANT1, PCB_ANT1, R1, R101_0Om1, RTC1, U7, U9
